Commit message: modified ocean_waves.world and added some seemingly unnecessary material files

File: uuv_sensor_plugins/uuv_sensor_ros_plugins/urdf/camera_snippets.xacro (robot description, xacro)
@@ -144,11 +144,13 @@
     params="namespace suffix parent_link topic mass update_rate
       hfov width height stddev
-      *inertia *origin">
+       *inertia *origin">
     <!-- Sensor link -->
     <link name="${namespace}/camera${suffix}_link">
       <inertial>
-        <xacro:insert_block name="inertia" />
+        <!--xacro:insert_block name="inertia" /-->
         <mass value="${mass}" />
+	<inertia ixx="0.00001" ixy="0.0" ixz="0.0" iyy="0.00001" iyz="0.0" izz="0.00001" />
         <origin xyz="0 0 0" rpy="0 0 0" />
+	 <!--xacro:insert_block name="origin" /-->
       </inertial>
       <visual>
@@ -160,5 +162,6 @@
     </link>
     <joint name="${namespace}/camera${suffix}_joint" type="revolute">
-      <xacro:insert_block name="origin" />
+      <!--xacro:insert_block name="origin" / -->
+      <origin xyz="1.4 0 -1" rpy="0 0.78 0"/>
       <parent link="${parent_link}" />
       <child link="${namespace}/camera${suffix}_link" />
@@ -206,5 +209,5 @@
           </noise>
         </camera>
-        <plugin name="camera${suffix}_controller" filename="libuuv_gazebo_ros_camera_plugin.so">
+        <!--plugin name="camera${suffix}_controller" filename="libuuv_gazebo_ros_camera_plugin.so">
           <updateRate>${update_rate}</updateRate>
           <cameraName>${namespace}/camera${suffix}</cameraName>
@@ -216,11 +219,39 @@
           <backgroundG>0</backgroundG>
           <backgroundB>0</backgroundB>
-          <!-- required for ros depth cam -->
-          <imageTopicName>${topic}_image</imageTopicName>
+          <required for ros depth cam -->
+          <!--imageTopicName>${topic}_image</imageTopicName>
           <pointCloudTopicName>${topic}_cloud</pointCloudTopicName>
           <depthImageTopicName>${topic}_depth</depthImageTopicName>
           <depthImageCameraInfoTopicName>${topic}_depth_info</depthImageCameraInfoTopicName>
           <pointCloudCutoff>10.0</pointCloudCutoff>
+        </plugin-->
+	<!--ALG Edit adding kinect depth camera -->
+	<plugin name="camera_plugin" filename="libgazebo_ros_openni_kinect.so">
+          <baseline>0.2</baseline>
+          <alwaysOn>true</alwaysOn>
+          <!-- Keep this zero, update_rate in the parent <sensor> tag
+            will control the frame rate. -->
+          <updateRate>0.0</updateRate>
+          <cameraName>camera_ir</cameraName>
+          <imageTopicName>/camera/color/image_raw</imageTopicName>
+          <cameraInfoTopicName>/camera/color/camera_info</cameraInfoTopicName>
+          <depthImageTopicName>/camera/depth/image_raw</depthImageTopicName>
+          <depthImageCameraInfoTopicName>/camera/depth/camera_info</depthImageCameraInfoTopicName>
+          <pointCloudTopicName>/camera/depth/points</pointCloudTopicName>
+          <frameName>cameradeepth_link</frameName>
+          <pointCloudCutoff>0.5</pointCloudCutoff>
+          <pointCloudCutoffMax>3.0</pointCloudCutoffMax>
+          <distortionK1>0</distortionK1>
+          <distortionK2>0</distortionK2>
+          <distortionK3>0</distortionK3>
+          <distortionT1>0</distortionT1>
+          <distortionT2>0</distortionT2>
+          <CxPrime>0</CxPrime>
+          <Cx>0</Cx>
+          <Cy>0</Cy>
+          <focalLength>0</focalLength>
+          <hackBaseline>0</hackBaseline>
         </plugin>
+	<!-- End of ALGEdit -->
       </sensor>
     </gazebo>

File: uuv_sensor_plugins/uuv_sensor_ros_plugins/urdf/stereo_snippets.xacro (robot description, xacro)
@@ -78,5 +78,6 @@
         <alwaysOn>true</alwaysOn>
         <updateRate>30.0</updateRate>
-        <cameraName>${namespace}/duo3d_left</cameraName>
+        <!--cameraName>${namespace}/duo3d_left</cameraName -->
+	<cameraName>left</cameraName>
         <imageTopicName>image_raw</imageTopicName>
         <cameraInfoTopicName>camera_info</cameraInfoTopicName>
@@ -133,8 +134,10 @@
         <alwaysOn>true</alwaysOn>
         <updateRate>30.0</updateRate>
-        <cameraName>${namespace}/duo3d_right</cameraName>
-        <imageTopicName>image_raw</imageTopicName>
+        <!--cameraName>${namespace}/duo3d_right</cameraName-->
+	<cameraName>right</cameraName>
+	<imageTopicName>image_raw</imageTopicName>
         <cameraInfoTopicName>camera_info</cameraInfoTopicName>
         <frameName>${namespace}/duo3d_right_link</frameName>
+	<!--frameName>rexrov2/duo3d_right_link</frameName-->
         <hackBaseline>0.07</hackBaseline>
         <distortionK1>${k1l}</distortionK1>
